Commit message: changed finger

File: models/franka_description/robots/panda_arm_hand_chopstick.urdf (robot description, URDF)
Before this commit: robot panda, 13 links, 12 joints
Links:
- link panda_leftfinger: geometry collision box size=0.01 0.004 0.08; visual box size=0.01 0.004 0.08
- link panda_rightfinger: geometry collision box size=0.01 0.004 0.08; visual box size=0.01 0.004 0.08
