Commit message: changed collision of hand

File: models/franka_description/robots/panda_arm_hand.urdf (robot description, URDF)
Before this commit: robot panda, 13 links, 12 joints
Links:
- link panda_hand: geometry collision box size=0.03 0.18 0.05; visual mesh filename=package://franka_description/meshes/visual/hand.dae
- link panda_leftfinger: geometry collision box size=0.01 0.004 0.06; visual mesh filename=package://franka_description/meshes/visual/finger.dae
- link panda_rightfinger: geometry collision box size=0.01 0.004 0.06; visual mesh filename=package://franka_description/meshes/visual/finger.dae

Commit message: smaller hand

File: models/franka_description/robots/panda_arm_hand.urdf (robot description, URDF)
Before this commit: robot panda, 13 links, 12 joints
Links:
- link panda_hand: geometry collision mesh filename=package://franka_description/meshes/collision/hand.stl scale=1 0.4 0.8; visual mesh filename=package://franka_description/meshes/visual/hand.dae scale=1 0.4 0.8
- link panda_leftfinger: geometry collision box size=0.01 0.004 0.08; visual box size=0.01 0.004 0.08
- link panda_link1: geometry visual mesh filename=package://franka_description/meshes/visual/link1.dae
- link panda_link2: geometry visual mesh filename=package://franka_description/meshes/visual/link2.dae
- link panda_link3: geometry visual mesh filename=package://franka_description/meshes/visual/link3.dae
- link panda_link4: geometry visual mesh filename=package://franka_description/meshes/visual/link4.dae
- link panda_link5: geometry visual mesh filename=package://franka_description/meshes/visual/link5.dae
- link panda_link6: geometry visual mesh filename=package://franka_description/meshes/visual/link6.dae
- link panda_link7: geometry visual mesh filename=package://franka_description/meshes/visual/link7.dae
- link panda_rightfinger: geometry collision box size=0.01 0.004 0.08; visual box size=0.01 0.004 0.08

Commit message: revolute 360 degree

File: models/franka_description/robots/panda_arm_hand.urdf (robot description, URDF)
Before this commit: robot panda, 13 links, 12 joints
Joints:
- joint panda_joint1: limit lower=-2.8973 upper=2.8973 effort=87 velocity=2.1750 -> effort=87 velocity=2.1750
- joint panda_joint3: limit lower=-2.8973 upper=2.8973 effort=87 velocity=2.1750 -> effort=87 velocity=2.1750
- joint panda_joint5: limit lower=-2.8973 upper=2.8973 effort=12 velocity=2.6100 -> effort=12 velocity=2.6100
- joint panda_joint7: limit lower=-2.8973 upper=2.8973 effort=12 velocity=2.6100 -> effort=12 velocity=2.6100

Commit message: rollback joint constraints

File: models/franka_description/robots/panda_arm_hand.urdf (robot description, URDF)
Before this commit: robot panda, 13 links, 12 joints
Joints:
- joint panda_joint1: limit effort=87 velocity=2.1750 -> lower=-2.8973 upper=2.8973 effort=87 velocity=2.1750
- joint panda_joint3: limit effort=87 velocity=2.1750 -> lower=-2.8973 upper=2.8973 effort=87 velocity=2.1750
- joint panda_joint5: limit effort=12 velocity=2.6100 -> lower=-2.8973 upper=2.8973 effort=12 velocity=2.6100
- joint panda_joint7: limit effort=12 velocity=2.6100 -> lower=-2.8973 upper=2.8973 effort=12 velocity=2.6100
